File: ArduinoFocuserPCB/ArduinoFocuserPCB.kicad_pcb (KiCad board)
At the start: 2 copper layers, 67.3 x 53.3 mm, 12 parts, among them M1 Stepper_Motor_bipolar, SW1 Rotary_Encoder_Switch, U1 DHT11

Commit message: git ignore
Parts:
- added U2: SN74HC14N, digikey-footprints:DIP-14_W3mm, F.Cu at (149.9, 50.8)
- moved U1 49.7 mm to (111.8, 77.5), turned to 180 degrees
- moved Motor1 16.6 mm to (125.7, 91.4), turned to 90 degrees
- moved C1 8.07 mm to (149.9, 90.2)
- moved R4 7.41 mm to (143.5, 52.1), turned to 270 degrees
- moved DRV1 6.35 mm to (153.7, 87.6)
- moved R1 4.58 mm to (143.5, 64.8), turned to 90 degrees
- moved C2 3.59 mm to (146.1, 62.2), turned to 270 degrees
- moved C3 2.82 mm to (146.1, 54.6), turned to 90 degrees
- moved R2 1.80 mm to (141.0, 64.8)
- moved R3 1.80 mm to (141.0, 52.1)
- moved SW1 1.80 mm to (137.2, 61.0)
- renumbered M1 to Motor1
Connections:
- A1 pad 20: ENCA -> ENCA_A
- A1 pad 21: ENCB -> ENCB_A
- A1 pad 23: DHTIO -> (no net)
- A1 pad 24: S1 -> S1_A
- A1 pad 28: (no net) -> DHTIO
Routing:
- net VCC: track 132.2 -> 185.4 mm
- net DHTIO: track 14.4 -> 44.9 mm
- net ENCA: track 31.4 -> 7.93 mm
- net ENCB: track 30.9 -> 7.93 mm
- net ENCA_A: track 0.00 -> 20.9 mm
- net ENCB_A: track 0.00 -> 14.8 mm
- net Net-(DRV1-Pad6): track 33.4 -> 45.4 mm
- net S1_A: track 0.00 -> 11.2 mm
- net Enable: track 41.1 -> 33.9 mm
- net Net-(DRV1-Pad5): track 35.9 -> 40.7 mm
- net M2: track 23.9 -> 19.6 mm
- net Net-(DRV1-Pad3): track 39.8 -> 35.7 mm
- net M1: track 22.9 -> 19.6 mm
- net Step: track 35.5 -> 32.9 mm
- net Dir: track 35.5 -> 32.9 mm
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Other:
- net class Power: clearance 1.016 -> 0.508; trace_width 1.016 -> 0.508; via_dia 1.016 -> 0.508
- board text added: "74HC14"
